Commit message: fixed the ompl bug. MoveIt planning is working

File: ros2_rm_robot/dual_rm_description/dual_rm_description/urdf/agv/woosh_agv.urdf.xacro (robot description, xacro)
@@ -309,5 +309,5 @@
     type="continuous">
     <origin
-      xyz="-0.148 0.015574 -0.153"
+      xyz="-0.148 0.015574 -0.16254"
       rpy="0 0 0" />
     <parent
@@ -325,5 +325,5 @@
     type="continuous">
     <origin
-      xyz="0.148 0.015574 -0.153"
+      xyz="0.148 0.015574 -0.16254"
       rpy="0 0 0" />
     <parent

File: ros2_rm_robot/dual_rm_description/dual_rm_description/urdf/arms/75b/left_arm.urdf.xacro (robot description, xacro)
@@ -147,5 +147,5 @@
     <xacro:visual_collision mesh="l_link6.STL" />
   </link>
-  <link
+  <!-- <link
     name="l_link7">
     <inertial>
@@ -162,7 +162,7 @@
         iyz="-1.7799E-08"
         izz="0.00035278" />
-    </inertial>
-    <xacro:visual_collision mesh="l_link7.STL" />
-  </link>
+    </inertial> -->
+    <!-- <xacro:visual_collision mesh="l_link7.STL" />
+  </link> -->
   <joint
     name="l_joint1"
@@ -273,5 +273,5 @@
       velocity="3.925" />
   </joint>
-  <joint
+  <!-- <joint
     name="l_joint7"
     type="revolute">
@@ -290,4 +290,4 @@
       effort="10"
       velocity="3.925" />
-  </joint>
+  </joint> -->
 </robot>

File: ros2_rm_robot/dual_rm_description/dual_rm_description/urdf/arms/75b/right_arm.urdf.xacro (robot description, xacro)
@@ -147,5 +147,5 @@
     <xacro:visual_collision mesh="r_link6.STL" />
   </link>
-  <link
+  <!-- <link
     name="r_link7">
     <inertial>
@@ -163,6 +163,6 @@
         izz="0.00035277" />
     </inertial>
-    <xacro:visual_collision mesh="r_link7.STL" />
-  </link>
+    <xacro:visual_collision mesh="r_link7.STL" /> -->
+  <!-- </link> -->
   <joint
     name="r_joint1"
@@ -273,5 +273,5 @@
       velocity="3.925" />
   </joint>
-  <joint
+  <!-- <joint
     name="r_joint7"
     type="revolute">
@@ -290,4 +290,4 @@
       effort="10"
       velocity="3.925" />
-  </joint>
+  </joint> -->
 </robot>

File: ros2_rm_robot/dual_rm_gazebo/config/dual_rm_75b_gazebo.urdf.xacro (robot description, xacro)
@@ -1,152 +1,181 @@
 <?xml version="1.0"?>
-<robot xmlns:xacro="http://www.ros.org/wiki/xacro" name="dual_rm_75b_gazebo">
-    <link name="world"/>
-    <joint name="fixed" type="fixed">
-        <parent link="world"/>
-        <child link="base_link_underpan"/>
-    </joint>
+<robot xmlns:xacro="http://www.ros.org/wiki/xacro" name="dual_rm_75b_description">
     <xacro:include filename="$(find dual_rm_75b_description)/urdf/dual_rm_75b_description.urdf.xacro" />
+    <!-- <xacro:include filename="$(find dual_rm_gazebo)/config/dg4f_gazebo_classic.urdf.xacro"/> -->
     <gazebo reference="base_link">
         <self_collide>false</self_collide>
-        <gravity>false</gravity>
+        <gravity>true</gravity>
     </gazebo>
     <gazebo reference="r_link1">
         <self_collide>false</self_collide>
-        <gravity>false</gravity>
+        <gravity>true</gravity>
     </gazebo>
     <gazebo reference="r_link2">
         <self_collide>false</self_collide>
-        <gravity>false</gravity>
+        <gravity>true</gravity>
     </gazebo>
     <gazebo reference="r_link3">
         <self_collide>false</self_collide>
-        <gravity>false</gravity>
+        <gravity>true</gravity>
     </gazebo>
     <gazebo reference="r_link4">
         <self_collide>false</self_collide>
-        <gravity>false</gravity>
+        <gravity>true</gravity>
     </gazebo>
     <gazebo reference="r_link5">
         <self_collide>false</self_collide>
-        <gravity>false</gravity>
+        <gravity>true</gravity>
     </gazebo>
     <gazebo reference="r_link6">
         <self_collide>false</self_collide>
-        <gravity>false</gravity>
-    </gazebo>
-    <gazebo reference="r_link7">
-        <self_collide>false</self_collide>
-        <gravity>false</gravity>
-    </gazebo>
+        <gravity>true</gravity>
+    </gazebo>
+    <!-- <gazebo reference="r_link7">
+        <self_collide>false</self_collide>
+        <gravity>true</gravity>
+    </gazebo> -->
     <gazebo reference="l_link1">
         <self_collide>false</self_collide>
-        <gravity>false</gravity>
+        <gravity>true</gravity>
     </gazebo>
     <gazebo reference="l_link2">
         <self_collide>false</self_collide>
-        <gravity>false</gravity>
+        <gravity>true</gravity>
     </gazebo>
     <gazebo reference="l_link3">
         <self_collide>false</self_collide>
-        <gravity>false</gravity>
+        <gravity>true</gravity>
     </gazebo>
     <gazebo reference="l_link4">
         <self_collide>false</self_collide>
-        <gravity>false</gravity>
+        <gravity>true</gravity>
     </gazebo>
     <gazebo reference="l_link5">
         <self_collide>false</self_collide>
-        <gravity>false</gravity>
+        <gravity>true</gravity>
     </gazebo>
     <gazebo reference="l_link6">
         <self_collide>false</self_collide>
-        <gravity>false</gravity>
-    </gazebo>
-    <gazebo reference="l_link7">
-        <self_collide>false</self_collide>
-        <gravity>false</gravity>
-    </gazebo>
+        <gravity>true</gravity>
+    </gazebo>
+    <!-- <gazebo reference="l_link7">
+        <self_collide>false</self_collide>
+        <gravity>true</gravity>
+    </gazebo> -->
     <gazebo reference="head_link1">
         <self_collide>false</self_collide>
-        <gravity>false</gravity>
+        <gravity>true</gravity>
     </gazebo>
     <gazebo reference="head_link2">
         <self_collide>false</self_collide>
-        <gravity>false</gravity>
+        <gravity>true</gravity>
     </gazebo>
     <gazebo reference="camera_link">
         <self_collide>false</self_collide>
-        <gravity>false</gravity>
+        <gravity>true</gravity>
     </gazebo>
     <gazebo reference="link_right_wheel">
         <self_collide>false</self_collide>
-        <gravity>false</gravity>
+        <gravity>true</gravity>
+        <mu1>10.0</mu1>
+        <mu2>10.0</mu2>
+        <kp>1000000.0</kp>
+        <kd>1.0</kd>
+        <minDepth>0.001</minDepth>
+        <maxVel>1.0</maxVel>
     </gazebo>
     <gazebo reference="link_left_wheel">
         <self_collide>false</self_collide>
-        <gravity>false</gravity>
+        <gravity>true</gravity>
+        <mu1>10.0</mu1>
+        <mu2>10.0</mu2>
+        <kp>1000000.0</kp>
+        <kd>1.0</kd>
+        <minDepth>0.001</minDepth>
+        <maxVel>1.0</maxVel>
     </gazebo>
     <gazebo reference="link_swivel_wheel_1_1">
         <self_collide>false</self_collide>
-        <gravity>false</gravity>
+        <gravity>true</gravity>
+        <mu1>0.0</mu1>
+        <mu2>0.0</mu2>
     </gazebo>
     <gazebo reference="link_swivel_wheel_1_2">
         <self_collide>false</self_collide>
-        <gravity>false</gravity>
+        <gravity>true</gravity>
+        <mu1>0.0</mu1>
+        <mu2>0.0</mu2>
     </gazebo>
     <gazebo reference="link_swivel_wheel_2_1">
         <self_collide>false</self_collide>
-        <gravity>false</gravity>
+        <gravity>true</gravity>
+        <mu1>0.0</mu1>
+        <mu2>0.0</mu2>
     </gazebo>
     <gazebo reference="link_swivel_wheel_2_2">
         <self_collide>false</self_collide>
-        <gravity>false</gravity>
+        <gravity>true</gravity>
+        <mu1>0.0</mu1>
+        <mu2>0.0</mu2>
     </gazebo>
     <gazebo reference="link_swivel_wheel_3_1">
         <self_collide>false</self_collide>
-        <gravity>false</gravity>
+        <gravity>true</gravity>
+        <mu1>0.0</mu1>
+        <mu2>0.0</mu2>
     </gazebo>
     <gazebo reference="link_swivel_wheel_3_2">
         <self_collide>false</self_collide>
-        <gravity>false</gravity>
+        <gravity>true</gravity>
+        <mu1>0.0</mu1>
+        <mu2>0.0</mu2>
     </gazebo>
     <gazebo reference="link_swivel_wheel_4_1">
         <self_collide>false</self_collide>
-        <gravity>false</gravity>
+        <gravity>true</gravity>
+        <mu1>0.0</mu1>
+        <mu2>0.0</mu2>
     </gazebo>
     <gazebo reference="link_swivel_wheel_4_2">
         <self_collide>false</self_collide>
-        <gravity>false</gravity>
+        <gravity>true</gravity>
+        <mu1>0.0</mu1>
+        <mu2>0.0</mu2>
     </gazebo>
     <gazebo reference="body_base_link">
         <self_collide>false</self_collide>
-        <gravity>false</gravity>
+        <gravity>true</gravity>
     </gazebo>
     <gazebo reference="platform_base_link">
         <self_collide>false</self_collide>
-        <gravity>false</gravity>
+        <gravity>true</gravity>
     </gazebo>
     <gazebo reference="l_base_link1">
         <self_collide>false</self_collide>
-        <gravity>false</gravity>
+        <gravity>true</gravity>
     </gazebo>
     <gazebo reference="r_base_link1">
         <self_collide>false</self_collide>
-        <gravity>false</gravity>
+        <gravity>true</gravity>
     </gazebo>
     <gazebo reference="r_hand_base_link">
         <self_collide>false</self_collide>
-        <gravity>false</gravity>
+        <gravity>true</gravity>
     </gazebo>
     <gazebo reference="l_hand_base_link">
         <self_collide>false</self_collide>
-        <gravity>false</gravity>
+        <gravity>true</gravity>
     </gazebo>
     <gazebo reference="base_link_underpan">
         <self_collide>false</self_collide>
-        <gravity>false</gravity>
-    </gazebo>
+        <gravity>true</gravity>
+    </gazebo>
+    <!-- <xacro:dg4f_attach
+        parent="l_hand_link"
+        xyz="0 0 0.01"
+        rpy="0 0 0"/>
+     -->
     <gazebo>
-        <is_static>true</is_static>
+        <is_static>false</is_static>
         <self_collide>true</self_collide>
     </gazebo>
@@ -275,5 +304,5 @@
         </joint>
         <joint name="joint_right_wheel">
-            <command_interface name="position"/>
+            <command_interface name="velocity"/>
             <state_interface name="position">
                 <param name="initial_value">0</param>
@@ -282,5 +311,5 @@
         </joint>
         <joint name="joint_left_wheel">
-            <command_interface name="position"/>
+            <command_interface name="velocity"/>
             <state_interface name="position">
                 <param name="initial_value">0</param>
@@ -289,5 +318,5 @@
         </joint>
         <joint name="joint_swivel_wheel_1_1">
-            <command_interface name="position"/>
+            <command_interface name="velocity"/>
             <state_interface name="position">
                 <param name="initial_value">0</param>
@@ -296,5 +325,5 @@
         </joint>
         <joint name="joint_swivel_wheel_1_2">
-            <command_interface name="position"/>
+            <command_interface name="velocity"/>
             <state_interface name="position">
                 <param name="initial_value">0</param>
@@ -303,5 +332,5 @@
         </joint>
         <joint name="joint_swivel_wheel_2_1">
-            <command_interface name="position"/>
+            <command_interface name="velocity"/>
             <state_interface name="position">
                 <param name="initial_value">0</param>
@@ -310,5 +339,5 @@
         </joint>
         <joint name="joint_swivel_wheel_2_2">
-            <command_interface name="position"/>
+            <command_interface name="velocity"/>
             <state_interface name="position">
                 <param name="initial_value">0</param>
@@ -317,5 +346,5 @@
         </joint>
         <joint name="joint_swivel_wheel_3_1">
-            <command_interface name="position"/>
+            <command_interface name="velocity"/>
             <state_interface name="position">
                 <param name="initial_value">0</param>
@@ -324,5 +353,5 @@
         </joint>
         <joint name="joint_swivel_wheel_3_2">
-            <command_interface name="position"/>
+            <command_interface name="velocity"/>
             <state_interface name="position">
                 <param name="initial_value">0</param>
@@ -331,5 +360,5 @@
         </joint>
         <joint name="joint_swivel_wheel_4_1">
-            <command_interface name="position"/>
+            <command_interface name="velocity"/>
             <state_interface name="position">
                 <param name="initial_value">0</param>
@@ -338,5 +367,5 @@
         </joint>
         <joint name="joint_swivel_wheel_4_2">
-            <command_interface name="position"/>
+            <command_interface name="velocity"/>
             <state_interface name="position">
                 <param name="initial_value">0</param>

File: ros2_rm_robot/dual_rm_moveit_config/dual_rm_75b_moveit_config/config/dual_rm_75b_description.ros2_control.xacro (robot description, xacro)
@@ -6,5 +6,5 @@
             <hardware>
                 <!-- By default, set up controllers for simulation. This won't work on real hardware -->
-                <plugin>mock_components/GenericSystem</plugin>
+                <plugin>fake_components/GenericSystem</plugin>
             </hardware>
             <joint name="l_joint1">
@@ -50,8 +50,15 @@
                 <state_interface name="velocity"/>
             </joint>
-            <joint name="l_joint7">
+            <!-- <joint name="l_joint7">
                 <command_interface name="position"/>
                 <state_interface name="position">
                   <param name="initial_value">${initial_positions['l_joint7']}</param>
+                </state_interface>
+                <state_interface name="velocity"/>
+            </joint> -->
+            <joint name="l_4c2_gripper_joint">
+                <command_interface name="position"/>
+                <state_interface name="position">
+                  <param name="initial_value">${initial_positions['l_4c2_gripper_joint']}</param>
                 </state_interface>
                 <state_interface name="velocity"/>
@@ -99,8 +106,15 @@
                 <state_interface name="velocity"/>
             </joint>
-            <joint name="r_joint7">
+            <!-- <joint name="r_joint7">
                 <command_interface name="position"/>
                 <state_interface name="position">
                   <param name="initial_value">${initial_positions['r_joint7']}</param>
+                </state_interface>
+                <state_interface name="velocity"/>
+            </joint> -->
+            <joint name="r_4c2_gripper_joint">
+                <command_interface name="position"/>
+                <state_interface name="position">
+                  <param name="initial_value">${initial_positions['r_4c2_gripper_joint']}</param>
                 </state_interface>
                 <state_interface name="velocity"/>
@@ -113,79 +127,4 @@
                 <state_interface name="velocity"/>
             </joint>
-            <!-- Passive joints: head and AGV wheels (state only, no command interface).
-                 These must be present so joint_state_broadcaster publishes their state
-                 and MoveIt's planning_scene_monitor sees the complete robot state. -->
-            <joint name="head_joint1">
-                <state_interface name="position">
-                  <param name="initial_value">0.0</param>
-                </state_interface>
-                <state_interface name="velocity"/>
-            </joint>
-            <joint name="head_joint2">
-                <state_interface name="position">
-                  <param name="initial_value">0.0</param>
-                </state_interface>
-                <state_interface name="velocity"/>
-            </joint>
-            <joint name="joint_left_wheel">
-                <state_interface name="position">
-                  <param name="initial_value">0.0</param>
-                </state_interface>
-                <state_interface name="velocity"/>
-            </joint>
-            <joint name="joint_right_wheel">
-                <state_interface name="position">
-                  <param name="initial_value">0.0</param>
-                </state_interface>
-                <state_interface name="velocity"/>
-            </joint>
-            <joint name="joint_swivel_wheel_1_1">
-                <state_interface name="position">
-                  <param name="initial_value">0.0</param>
-                </state_interface>
-                <state_interface name="velocity"/>
-            </joint>
-            <joint name="joint_swivel_wheel_1_2">
-                <state_interface name="position">
-                  <param name="initial_value">0.0</param>
-                </state_interface>
-                <state_interface name="velocity"/>
-            </joint>
-            <joint name="joint_swivel_wheel_2_1">
-                <state_interface name="position">
-                  <param name="initial_value">0.0</param>
-                </state_interface>
-                <state_interface name="velocity"/>
-            </joint>
-            <joint name="joint_swivel_wheel_2_2">
-                <state_interface name="position">
-                  <param name="initial_value">0.0</param>
-                </state_interface>
-                <state_interface name="velocity"/>
-            </joint>
-            <joint name="joint_swivel_wheel_3_1">
-                <state_interface name="position">
-                  <param name="initial_value">0.0</param>
-                </state_interface>
-                <state_interface name="velocity"/>
-            </joint>
-            <joint name="joint_swivel_wheel_3_2">
-                <state_interface name="position">
-                  <param name="initial_value">0.0</param>
-                </state_interface>
-                <state_interface name="velocity"/>
-            </joint>
-            <joint name="joint_swivel_wheel_4_1">
-                <state_interface name="position">
-                  <param name="initial_value">0.0</param>
-                </state_interface>
-                <state_interface name="velocity"/>
-            </joint>
-            <joint name="joint_swivel_wheel_4_2">
-                <state_interface name="position">
-                  <param name="initial_value">0.0</param>
-                </state_interface>
-                <state_interface name="velocity"/>
-            </joint>
         </ros2_control>
     </xacro:macro>

File: ros2_rm_robot/dual_rm_moveit_config/dual_rm_75b_moveit_config/config/dual_rm_75b_description.urdf.xacro (robot description, xacro)
@@ -2,7 +2,6 @@
 <robot xmlns:xacro="http://www.ros.org/wiki/xacro" name="dual_rm_75b_description">
     <xacro:arg name="initial_positions_file" default="initial_positions.yaml" />
-    <!-- Import robot description (unified package, 75b variant) -->
-    <xacro:arg name="arm_model" default="75b"/>
-    <xacro:include filename="$(find dual_rm_description)/urdf/r2d3_description.urdf.xacro" />
+    <!-- Import dual_rm_75b_description urdf file -->
+    <xacro:include filename="$(find dual_rm_75b_description)/urdf/dual_rm_75b_description.urdf.xacro" />
     <!-- Import control_xacro -->
     <xacro:include filename="dual_rm_75b_description.ros2_control.xacro" />
