Commit message: Bringup launch works for all cases of both arm configuration with both grippers with help of arguments

File: ros2_rm_robot/dual_rm_description/dual_rm_description/urdf/agv/woosh_agv.urdf.xacro (robot description, xacro)
@@ -309,5 +309,5 @@
     type="continuous">
     <origin
-      xyz="-0.148 0.015574 -0.16254"
+      xyz="-0.148 0.015574 -0.153"
       rpy="0 0 0" />
     <parent
@@ -325,5 +325,5 @@
     type="continuous">
     <origin
-      xyz="0.148 0.015574 -0.16254"
+      xyz="0.148 0.015574 -0.153"
       rpy="0 0 0" />
     <parent

File: ros2_rm_robot/dual_rm_description/dual_rm_description/urdf/arms/65b/joints.urdf.xacro (robot description, xacro)
@@ -43,39 +43,42 @@
       xyz="0 0 0" />
   </joint>
-  <joint
-    name="r_hand_joint"
-    type="fixed">
-    <origin
-      xyz="0 0 0.0445"
-      rpy="0 0 0" />
-    <parent
-      link="r_link6" />
-    <child
-      link="r_hand_base_link" />
-    <axis
-      xyz="0 0 -1" />
-    <limit
-      lower="0"
-      upper="0"
-      effort="0"
-      velocity="0" />
-  </joint>
-  <joint
-    name="l_hand_joint"
-    type="fixed">
-    <origin
-      xyz="0 0 0.0445"
-      rpy="3.1415 3.1415 3.1415" />
-    <parent
-      link="l_link6" />
-    <child
-      link="l_hand_base_link" />
-    <axis
-      xyz="0 0 0" />
-    <limit
-      lower="0"
-      upper="0"
-      effort="0"
-      velocity="0" />
-  </joint>
+  <!-- Dummy Hand Joints Wrapped in Conditional -->
+  <xacro:if value="${gripper_type == 'dummy'}">
+    <joint
+      name="r_hand_joint"
+      type="fixed">
+      <origin
+        xyz="0 0 0.0445"
+        rpy="0 0 0" />
+      <parent
+        link="r_link6" />
+      <child
+        link="r_hand_base_link" />
+      <axis
+        xyz="0 0 -1" />
+      <limit
+        lower="0"
+        upper="0"
+        effort="0"
+        velocity="0" />
+    </joint>
+    <joint
+      name="l_hand_joint"
+      type="fixed">
+      <origin
+        xyz="0 0 0.0445"
+        rpy="3.1415 3.1415 3.1415" />
+      <parent
+        link="l_link6" />
+      <child
+        link="l_hand_base_link" />
+      <axis
+        xyz="0 0 0" />
+      <limit
+        lower="0"
+        upper="0"
+        effort="0"
+        velocity="0" />
+    </joint>
+  </xacro:if>
 </robot>

File: ros2_rm_robot/dual_rm_description/dual_rm_description/urdf/arms/75b/joints.urdf.xacro (robot description, xacro)
@@ -43,39 +43,42 @@
       xyz="0 0 0" />
   </joint>
-  <!-- <joint
-    name="r_hand_joint"
-    type="fixed">
-    <origin
-      xyz="0 0 0.0445"
-      rpy="0 0 0" />
-    <parent
-      link="r_link7" />
-    <child
-      link="r_hand" />
-    <axis
-      xyz="0 0 -1" />
-    <limit
-      lower="0"
-      upper="0"
-      effort="0"
-      velocity="0" />
-  </joint> -->
-  <!-- <joint
-    name="l_hand_joint"
-    type="fixed">
-    <origin
-      xyz="0 0 0.0445"
-      rpy="0 0 3.1415" />
-    <parent
-      link="l_link7" />
-    <child
-      link="l_hand_link" />
-    <axis
-      xyz="0 0 0" />
-    <limit
-      lower="0"
-      upper="0"
-      effort="0"
-      velocity="0" />
-  </joint>   -->
+  <!-- Dummy Hand Joints Wrapped in Conditional -->
+  <xacro:if value="${gripper_type == 'dummy'}">
+    <joint
+      name="r_hand_joint"
+      type="fixed">
+      <origin
+        xyz="0 0 0.0445"
+        rpy="0 0 0" />
+      <parent
+        link="r_link7" />
+      <child
+        link="r_hand" />
+      <axis
+        xyz="0 0 -1" />
+      <limit
+        lower="0"
+        upper="0"
+        effort="0"
+        velocity="0" />
+    </joint>
+    <joint
+      name="l_hand_joint"
+      type="fixed">
+      <origin
+        xyz="0 0 0.0445"
+        rpy="0 0 3.1415" />
+      <parent
+        link="l_link7" />
+      <child
+        link="l_hand_link" />
+      <axis
+        xyz="0 0 0" />
+      <limit
+        lower="0"
+        upper="0"
+        effort="0"
+        velocity="0" />
+    </joint>
+  </xacro:if>
 </robot>

File: ros2_rm_robot/dual_rm_description/dual_rm_description/urdf/arms/75b/left_arm.urdf.xacro (robot description, xacro)
@@ -147,5 +147,5 @@
     <xacro:visual_collision mesh="l_link6.STL" />
   </link>
-  <!-- <link
+  <link
     name="l_link7">
     <inertial>
@@ -162,7 +162,7 @@
         iyz="-1.7799E-08"
         izz="0.00035278" />
-    </inertial> -->
-    <!-- <xacro:visual_collision mesh="l_link7.STL" />
-  </link> -->
+    </inertial>
+    <xacro:visual_collision mesh="l_link7.STL" />
+  </link>
   <joint
     name="l_joint1"
@@ -273,5 +273,5 @@
       velocity="3.925" />
   </joint>
-  <!-- <joint
+  <joint
     name="l_joint7"
     type="revolute">
@@ -290,4 +290,4 @@
       effort="10"
       velocity="3.925" />
-  </joint> -->
+  </joint>
 </robot>

File: ros2_rm_robot/dual_rm_description/dual_rm_description/urdf/arms/75b/left_arm_transmission.xacro (robot description, xacro)
@@ -18,4 +18,4 @@
   <xacro:rm75_b_v_left_transmission joint_name="l_joint5" />
   <xacro:rm75_b_v_left_transmission joint_name="l_joint6" />
-  <!-- <xacro:rm75_b_v_left_transmission joint_name="l_joint7" /> -->
+  <xacro:rm75_b_v_left_transmission joint_name="l_joint7" />
 </robot>

File: ros2_rm_robot/dual_rm_description/dual_rm_description/urdf/arms/75b/right_arm.urdf.xacro (robot description, xacro)
@@ -147,5 +147,5 @@
     <xacro:visual_collision mesh="r_link6.STL" />
   </link>
-  <!-- <link
+  <link
     name="r_link7">
     <inertial>
@@ -163,6 +163,6 @@
         izz="0.00035277" />
     </inertial>
-    <xacro:visual_collision mesh="r_link7.STL" /> -->
-  <!-- </link> -->
+    <xacro:visual_collision mesh="r_link7.STL" />
+  </link>
   <joint
     name="r_joint1"
@@ -273,5 +273,5 @@
       velocity="3.925" />
   </joint>
-  <!-- <joint
+  <joint
     name="r_joint7"
     type="revolute">
@@ -290,4 +290,4 @@
       effort="10"
       velocity="3.925" />
-  </joint> -->
+  </joint>
 </robot>

File: ros2_rm_robot/dual_rm_description/dual_rm_description/urdf/arms/75b/right_arm_transmission.xacro (robot description, xacro)
@@ -18,4 +18,4 @@
   <xacro:rm75_b_v_right_transmission joint_name="r_joint5" />
   <xacro:rm75_b_v_right_transmission joint_name="r_joint6" />
-  <!-- <xacro:rm75_b_v_right_transmission joint_name="r_joint7" /> -->
+  <xacro:rm75_b_v_right_transmission joint_name="r_joint7" />
 </robot>

File: ros2_rm_robot/dual_rm_description/dual_rm_description/urdf/r2d3_description.urdf.xacro (robot description, xacro)
@@ -1,25 +1,48 @@
 <?xml version="1.0"?>
 <robot name="r2d3_description" xmlns:xacro="http://ros.org/wiki/xacro">
-    <xacro:arg name="arm_model" default="65b"/>
-    <xacro:property name="arm_model" value="$(arg arm_model)"/>
-    <!-- ═══════════════════════════════════════════════════════════
-         Shared components (identical for both arm variants)
-         ═══════════════════════════════════════════════════════════ -->
-    <xacro:include filename="$(find dual_rm_description)/urdf/materials/colors.urdf.xacro"/>
-    <xacro:include filename="$(find dual_rm_description)/urdf/agv/woosh_agv.urdf.xacro"/>
-    <xacro:include filename="$(find dual_rm_description)/urdf/body/body_head_platform.urdf.xacro"/>
-    <!-- ═══════════════════════════════════════════════════════════
-         Arm-variant components (selected by arm_model argument)
-         ═══════════════════════════════════════════════════════════ -->
-    <xacro:include filename="$(find dual_rm_description)/urdf/arms/$(arg arm_model)/left_arm.urdf.xacro"/>
+  <!-- TEMPORARILY CHANGE THESE DEFAULTS FOR THE SETUP ASSISTANT -->
+  <xacro:arg name="arm_model" default="65b"/>
+  <xacro:property name="arm_model" value="$(arg arm_model)"/>
+  <xacro:arg name="gripper_type" default="4c2"/>
+  <xacro:property name="gripper_type" value="$(arg gripper_type)"/>
+  <!-- ======================================================= -->
+  <!-- Shared components (identical for both arm variants)     -->
+  <!-- ======================================================= -->
+  <xacro:include filename="$(find dual_rm_description)/urdf/materials/colors.urdf.xacro"/>
+  <xacro:include filename="$(find dual_rm_description)/urdf/agv/woosh_agv.urdf.xacro"/>
+  <xacro:include filename="$(find dual_rm_description)/urdf/body/body_head_platform.urdf.xacro"/>
+  <!-- ======================================================= -->
+  <!-- Arm-variant components (selected by arm_model argument) -->
+  <!-- ======================================================= -->
+  <xacro:include filename="$(find dual_rm_description)/urdf/arms/$(arg arm_model)/left_arm.urdf.xacro"/>
+  <xacro:include filename="$(find dual_rm_description)/urdf/arms/$(arg arm_model)/right_arm.urdf.xacro"/>
+  <xacro:include filename="$(find dual_rm_description)/urdf/arms/$(arg arm_model)/joints.urdf.xacro"/>
+  <!-- ======================================================= -->
+  <!-- Gripper Selection                                       -->
+  <!-- ======================================================= -->
+  <xacro:if value="${gripper_type == 'dummy'}">
+    <!-- Load the original dummy hands -->
     <xacro:include filename="$(find dual_rm_description)/urdf/arms/$(arg arm_model)/left_hand.urdf.xacro"/>
-    <xacro:include filename="$(find dual_rm_description)/urdf/arms/$(arg arm_model)/right_arm.urdf.xacro"/>
     <xacro:include filename="$(find dual_rm_description)/urdf/arms/$(arg arm_model)/right_hand.urdf.xacro"/>
-    <xacro:include filename="$(find dual_rm_description)/urdf/arms/$(arg arm_model)/joints.urdf.xacro"/>
-    <!-- ═══════════════════════════════════════════════════════════
-         Transmissions (Only Useful For Gazebo Classic)
-         ═══════════════════════════════════════════════════════════ -->
-    <xacro:include filename="$(find dual_rm_description)/urdf/transmissions/body_head_platform_transmission.xacro"/>
-    <xacro:include filename="$(find dual_rm_description)/urdf/arms/$(arg arm_model)/left_arm_transmission.xacro"/>
-    <xacro:include filename="$(find dual_rm_description)/urdf/arms/$(arg arm_model)/right_arm_transmission.xacro"/>
+  </xacro:if>
+  <xacro:if value="${gripper_type == '4c2'}">
+    <!-- Load the new 4c2 Gripper Macro -->
+    <xacro:include filename="$(find dual_rm_description)/urdf/grippers/4c2_gripper.urdf.xacro"/>
+    <!-- Attach to the 6th link for the 65b model -->
+    <xacro:if value="${arm_model == '65b'}">
+      <xacro:gripper_4c2 prefix="l_" parent_link="l_link6" />
+      <xacro:gripper_4c2 prefix="r_" parent_link="r_link6" />
+    </xacro:if>
+    <!-- Attach to the 7th link for the 75b model -->
+    <xacro:if value="${arm_model == '75b'}">
+      <xacro:gripper_4c2 prefix="l_" parent_link="l_link7" />
+      <xacro:gripper_4c2 prefix="r_" parent_link="r_link7" />
+    </xacro:if>
+  </xacro:if>
+  <!-- ======================================================= -->
+  <!-- Transmissions (Only Useful For Gazebo Classic)          -->
+  <!-- ======================================================= -->
+  <xacro:include filename="$(find dual_rm_description)/urdf/transmissions/body_head_platform_transmission.xacro"/>
+  <xacro:include filename="$(find dual_rm_description)/urdf/arms/$(arg arm_model)/left_arm_transmission.xacro"/>
+  <xacro:include filename="$(find dual_rm_description)/urdf/arms/$(arg arm_model)/right_arm_transmission.xacro"/>
 </robot>

File: ros2_rm_robot/dual_rm_gazebo/config/dual_rm_75b_gazebo.urdf.xacro (robot description, xacro)
@@ -1,181 +1,152 @@
 <?xml version="1.0"?>
-<robot xmlns:xacro="http://www.ros.org/wiki/xacro" name="dual_rm_75b_description">
+<robot xmlns:xacro="http://www.ros.org/wiki/xacro" name="dual_rm_75b_gazebo">
+    <link name="world"/>
+    <joint name="fixed" type="fixed">
+        <parent link="world"/>
+        <child link="base_link_underpan"/>
+    </joint>
     <xacro:include filename="$(find dual_rm_75b_description)/urdf/dual_rm_75b_description.urdf.xacro" />
-    <!-- <xacro:include filename="$(find dual_rm_gazebo)/config/dg4f_gazebo_classic.urdf.xacro"/> -->
     <gazebo reference="base_link">
         <self_collide>false</self_collide>
-        <gravity>true</gravity>
+        <gravity>false</gravity>
     </gazebo>
     <gazebo reference="r_link1">
         <self_collide>false</self_collide>
-        <gravity>true</gravity>
+        <gravity>false</gravity>
     </gazebo>
     <gazebo reference="r_link2">
         <self_collide>false</self_collide>
-        <gravity>true</gravity>
+        <gravity>false</gravity>
     </gazebo>
     <gazebo reference="r_link3">
         <self_collide>false</self_collide>
-        <gravity>true</gravity>
+        <gravity>false</gravity>
     </gazebo>
     <gazebo reference="r_link4">
         <self_collide>false</self_collide>
-        <gravity>true</gravity>
+        <gravity>false</gravity>
     </gazebo>
     <gazebo reference="r_link5">
         <self_collide>false</self_collide>
-        <gravity>true</gravity>
+        <gravity>false</gravity>
     </gazebo>
     <gazebo reference="r_link6">
         <self_collide>false</self_collide>
-        <gravity>true</gravity>
-    </gazebo>
-    <!-- <gazebo reference="r_link7">
-        <self_collide>false</self_collide>
-        <gravity>true</gravity>
-    </gazebo> -->
+        <gravity>false</gravity>
+    </gazebo>
+    <gazebo reference="r_link7">
+        <self_collide>false</self_collide>
+        <gravity>false</gravity>
+    </gazebo>
     <gazebo reference="l_link1">
         <self_collide>false</self_collide>
-        <gravity>true</gravity>
+        <gravity>false</gravity>
     </gazebo>
     <gazebo reference="l_link2">
         <self_collide>false</self_collide>
-        <gravity>true</gravity>
+        <gravity>false</gravity>
     </gazebo>
     <gazebo reference="l_link3">
         <self_collide>false</self_collide>
-        <gravity>true</gravity>
+        <gravity>false</gravity>
     </gazebo>
     <gazebo reference="l_link4">
         <self_collide>false</self_collide>
-        <gravity>true</gravity>
+        <gravity>false</gravity>
     </gazebo>
     <gazebo reference="l_link5">
         <self_collide>false</self_collide>
-        <gravity>true</gravity>
+        <gravity>false</gravity>
     </gazebo>
     <gazebo reference="l_link6">
         <self_collide>false</self_collide>
-        <gravity>true</gravity>
-    </gazebo>
-    <!-- <gazebo reference="l_link7">
-        <self_collide>false</self_collide>
-        <gravity>true</gravity>
-    </gazebo> -->
+        <gravity>false</gravity>
+    </gazebo>
+    <gazebo reference="l_link7">
+        <self_collide>false</self_collide>
+        <gravity>false</gravity>
+    </gazebo>
     <gazebo reference="head_link1">
         <self_collide>false</self_collide>
-        <gravity>true</gravity>
+        <gravity>false</gravity>
     </gazebo>
     <gazebo reference="head_link2">
         <self_collide>false</self_collide>
-        <gravity>true</gravity>
+        <gravity>false</gravity>
     </gazebo>
     <gazebo reference="camera_link">
         <self_collide>false</self_collide>
-        <gravity>true</gravity>
+        <gravity>false</gravity>
     </gazebo>
     <gazebo reference="link_right_wheel">
         <self_collide>false</self_collide>
-        <gravity>true</gravity>
-        <mu1>10.0</mu1>
-        <mu2>10.0</mu2>
-        <kp>1000000.0</kp>
-        <kd>1.0</kd>
-        <minDepth>0.001</minDepth>
-        <maxVel>1.0</maxVel>
+        <gravity>false</gravity>
     </gazebo>
     <gazebo reference="link_left_wheel">
         <self_collide>false</self_collide>
-        <gravity>true</gravity>
-        <mu1>10.0</mu1>
-        <mu2>10.0</mu2>
-        <kp>1000000.0</kp>
-        <kd>1.0</kd>
-        <minDepth>0.001</minDepth>
-        <maxVel>1.0</maxVel>
+        <gravity>false</gravity>
     </gazebo>
     <gazebo reference="link_swivel_wheel_1_1">
         <self_collide>false</self_collide>
-        <gravity>true</gravity>
-        <mu1>0.0</mu1>
-        <mu2>0.0</mu2>
+        <gravity>false</gravity>
     </gazebo>
     <gazebo reference="link_swivel_wheel_1_2">
         <self_collide>false</self_collide>
-        <gravity>true</gravity>
-        <mu1>0.0</mu1>
-        <mu2>0.0</mu2>
+        <gravity>false</gravity>
     </gazebo>
     <gazebo reference="link_swivel_wheel_2_1">
         <self_collide>false</self_collide>
-        <gravity>true</gravity>
-        <mu1>0.0</mu1>
-        <mu2>0.0</mu2>
+        <gravity>false</gravity>
     </gazebo>
     <gazebo reference="link_swivel_wheel_2_2">
         <self_collide>false</self_collide>
-        <gravity>true</gravity>
-        <mu1>0.0</mu1>
-        <mu2>0.0</mu2>
+        <gravity>false</gravity>
     </gazebo>
     <gazebo reference="link_swivel_wheel_3_1">
         <self_collide>false</self_collide>
-        <gravity>true</gravity>
-        <mu1>0.0</mu1>
-        <mu2>0.0</mu2>
+        <gravity>false</gravity>
     </gazebo>
     <gazebo reference="link_swivel_wheel_3_2">
         <self_collide>false</self_collide>
-        <gravity>true</gravity>
-        <mu1>0.0</mu1>
-        <mu2>0.0</mu2>
+        <gravity>false</gravity>
     </gazebo>
     <gazebo reference="link_swivel_wheel_4_1">
         <self_collide>false</self_collide>
-        <gravity>true</gravity>
-        <mu1>0.0</mu1>
-        <mu2>0.0</mu2>
+        <gravity>false</gravity>
     </gazebo>
     <gazebo reference="link_swivel_wheel_4_2">
         <self_collide>false</self_collide>
-        <gravity>true</gravity>
-        <mu1>0.0</mu1>
-        <mu2>0.0</mu2>
+        <gravity>false</gravity>
     </gazebo>
     <gazebo reference="body_base_link">
         <self_collide>false</self_collide>
-        <gravity>true</gravity>
+        <gravity>false</gravity>
     </gazebo>
     <gazebo reference="platform_base_link">
         <self_collide>false</self_collide>
-        <gravity>true</gravity>
+        <gravity>false</gravity>
     </gazebo>
     <gazebo reference="l_base_link1">
         <self_collide>false</self_collide>
-        <gravity>true</gravity>
+        <gravity>false</gravity>
     </gazebo>
     <gazebo reference="r_base_link1">
         <self_collide>false</self_collide>
-        <gravity>true</gravity>
+        <gravity>false</gravity>
     </gazebo>
     <gazebo reference="r_hand_base_link">
         <self_collide>false</self_collide>
-        <gravity>true</gravity>
+        <gravity>false</gravity>
     </gazebo>
     <gazebo reference="l_hand_base_link">
         <self_collide>false</self_collide>
-        <gravity>true</gravity>
+        <gravity>false</gravity>
     </gazebo>
     <gazebo reference="base_link_underpan">
         <self_collide>false</self_collide>
-        <gravity>true</gravity>
-    </gazebo>
-    <!-- <xacro:dg4f_attach
-        parent="l_hand_link"
-        xyz="0 0 0.01"
-        rpy="0 0 0"/>
-     -->
+        <gravity>false</gravity>
+    </gazebo>
     <gazebo>
-        <is_static>false</is_static>
+        <is_static>true</is_static>
         <self_collide>true</self_collide>
     </gazebo>
@@ -304,5 +275,5 @@
         </joint>
         <joint name="joint_right_wheel">
-            <command_interface name="velocity"/>
+            <command_interface name="position"/>
             <state_interface name="position">
                 <param name="initial_value">0</param>
@@ -311,5 +282,5 @@
         </joint>
         <joint name="joint_left_wheel">
-            <command_interface name="velocity"/>
+            <command_interface name="position"/>
             <state_interface name="position">
                 <param name="initial_value">0</param>
@@ -318,5 +289,5 @@
         </joint>
         <joint name="joint_swivel_wheel_1_1">
-            <command_interface name="velocity"/>
+            <command_interface name="position"/>
             <state_interface name="position">
                 <param name="initial_value">0</param>
@@ -325,5 +296,5 @@
         </joint>
         <joint name="joint_swivel_wheel_1_2">
-            <command_interface name="velocity"/>
+            <command_interface name="position"/>
             <state_interface name="position">
                 <param name="initial_value">0</param>
@@ -332,5 +303,5 @@
         </joint>
         <joint name="joint_swivel_wheel_2_1">
-            <command_interface name="velocity"/>
+            <command_interface name="position"/>
             <state_interface name="position">
                 <param name="initial_value">0</param>
@@ -339,5 +310,5 @@
         </joint>
         <joint name="joint_swivel_wheel_2_2">
-            <command_interface name="velocity"/>
+            <command_interface name="position"/>
             <state_interface name="position">
                 <param name="initial_value">0</param>
@@ -346,5 +317,5 @@
         </joint>
         <joint name="joint_swivel_wheel_3_1">
-            <command_interface name="velocity"/>
+            <command_interface name="position"/>
             <state_interface name="position">
                 <param name="initial_value">0</param>
@@ -353,5 +324,5 @@
         </joint>
         <joint name="joint_swivel_wheel_3_2">
-            <command_interface name="velocity"/>
+            <command_interface name="position"/>
             <state_interface name="position">
                 <param name="initial_value">0</param>
@@ -360,5 +331,5 @@
         </joint>
         <joint name="joint_swivel_wheel_4_1">
-            <command_interface name="velocity"/>
+            <command_interface name="position"/>
             <state_interface name="position">
                 <param name="initial_value">0</param>
@@ -367,5 +338,5 @@
         </joint>
         <joint name="joint_swivel_wheel_4_2">
-            <command_interface name="velocity"/>
+            <command_interface name="position"/>
             <state_interface name="position">
                 <param name="initial_value">0</param>
