Commit message: Bringup launch works for all cases of both arm configuration with both grippers with help of arguments

File: ros2_rm_robot/dual_rm_moveit_config/dual_rm_75b_moveit_config/config/dual_rm_75b_description.ros2_control.xacro (robot description, xacro)
@@ -6,5 +6,5 @@
             <hardware>
                 <!-- By default, set up controllers for simulation. This won't work on real hardware -->
-                <plugin>fake_components/GenericSystem</plugin>
+                <plugin>mock_components/GenericSystem</plugin>
             </hardware>
             <joint name="l_joint1">
@@ -50,15 +50,8 @@
                 <state_interface name="velocity"/>
             </joint>
-            <!-- <joint name="l_joint7">
+            <joint name="l_joint7">
                 <command_interface name="position"/>
                 <state_interface name="position">
                   <param name="initial_value">${initial_positions['l_joint7']}</param>
-                </state_interface>
-                <state_interface name="velocity"/>
-            </joint> -->
-            <joint name="l_4c2_gripper_joint">
-                <command_interface name="position"/>
-                <state_interface name="position">
-                  <param name="initial_value">${initial_positions['l_4c2_gripper_joint']}</param>
                 </state_interface>
                 <state_interface name="velocity"/>
@@ -106,15 +99,8 @@
                 <state_interface name="velocity"/>
             </joint>
-            <!-- <joint name="r_joint7">
+            <joint name="r_joint7">
                 <command_interface name="position"/>
                 <state_interface name="position">
                   <param name="initial_value">${initial_positions['r_joint7']}</param>
-                </state_interface>
-                <state_interface name="velocity"/>
-            </joint> -->
-            <joint name="r_4c2_gripper_joint">
-                <command_interface name="position"/>
-                <state_interface name="position">
-                  <param name="initial_value">${initial_positions['r_4c2_gripper_joint']}</param>
                 </state_interface>
                 <state_interface name="velocity"/>
@@ -127,4 +113,79 @@
                 <state_interface name="velocity"/>
             </joint>
+            <!-- Passive joints: head and AGV wheels (state only, no command interface).
+                 These must be present so joint_state_broadcaster publishes their state
+                 and MoveIt's planning_scene_monitor sees the complete robot state. -->
+            <joint name="head_joint1">
+                <state_interface name="position">
+                  <param name="initial_value">0.0</param>
+                </state_interface>
+                <state_interface name="velocity"/>
+            </joint>
+            <joint name="head_joint2">
+                <state_interface name="position">
+                  <param name="initial_value">0.0</param>
+                </state_interface>
+                <state_interface name="velocity"/>
+            </joint>
+            <joint name="joint_left_wheel">
+                <state_interface name="position">
+                  <param name="initial_value">0.0</param>
+                </state_interface>
+                <state_interface name="velocity"/>
+            </joint>
+            <joint name="joint_right_wheel">
+                <state_interface name="position">
+                  <param name="initial_value">0.0</param>
+                </state_interface>
+                <state_interface name="velocity"/>
+            </joint>
+            <joint name="joint_swivel_wheel_1_1">
+                <state_interface name="position">
+                  <param name="initial_value">0.0</param>
+                </state_interface>
+                <state_interface name="velocity"/>
+            </joint>
+            <joint name="joint_swivel_wheel_1_2">
+                <state_interface name="position">
+                  <param name="initial_value">0.0</param>
+                </state_interface>
+                <state_interface name="velocity"/>
+            </joint>
+            <joint name="joint_swivel_wheel_2_1">
+                <state_interface name="position">
+                  <param name="initial_value">0.0</param>
+                </state_interface>
+                <state_interface name="velocity"/>
+            </joint>
+            <joint name="joint_swivel_wheel_2_2">
+                <state_interface name="position">
+                  <param name="initial_value">0.0</param>
+                </state_interface>
+                <state_interface name="velocity"/>
+            </joint>
+            <joint name="joint_swivel_wheel_3_1">
+                <state_interface name="position">
+                  <param name="initial_value">0.0</param>
+                </state_interface>
+                <state_interface name="velocity"/>
+            </joint>
+            <joint name="joint_swivel_wheel_3_2">
+                <state_interface name="position">
+                  <param name="initial_value">0.0</param>
+                </state_interface>
+                <state_interface name="velocity"/>
+            </joint>
+            <joint name="joint_swivel_wheel_4_1">
+                <state_interface name="position">
+                  <param name="initial_value">0.0</param>
+                </state_interface>
+                <state_interface name="velocity"/>
+            </joint>
+            <joint name="joint_swivel_wheel_4_2">
+                <state_interface name="position">
+                  <param name="initial_value">0.0</param>
+                </state_interface>
+                <state_interface name="velocity"/>
+            </joint>
         </ros2_control>
     </xacro:macro>

File: ros2_rm_robot/dual_rm_moveit_config/dual_rm_75b_moveit_config/config/dual_rm_75b_description.urdf.xacro (robot description, xacro)
@@ -1,8 +1,11 @@
 <?xml version="1.0"?>
 <robot xmlns:xacro="http://www.ros.org/wiki/xacro" name="dual_rm_75b_description">
-    <xacro:arg name="initial_positions_file" default="initial_positions.yaml" />
-    <!-- Import dual_rm_75b_description urdf file -->
-    <xacro:include filename="$(find dual_rm_75b_description)/urdf/dual_rm_75b_description.urdf.xacro" />
-    <!-- Import control_xacro -->
+    <xacro:arg name="arm_model" default="75b"/>
+    <!-- ADD THIS LINE SO MOVEIT KNOWS ABOUT THE 4C2 -->
+    <xacro:arg name="gripper_type" default="4c2"/>
+    <xacro:arg name="initial_positions_file" default="initial_positions.yaml"/>
+    <!-- Import robot description -->
+    <xacro:include filename="$(find dual_rm_description)/urdf/r2d3_description.urdf.xacro" />
+    <!-- Import control xacro -->
     <xacro:include filename="dual_rm_75b_description.ros2_control.xacro" />
     <xacro:dual_rm_75b_description_ros2_control name="FakeSystem" initial_positions_file="$(arg initial_positions_file)"/>
