Commit message: Corrected testing files and added readme files

File: ros2_rm_robot/dual_rm_gazebo/config/dual_rm_65b_gazebo.urdf.xacro (robot description, xacro)
@@ -1,4 +1,5 @@
 <?xml version="1.0"?>
 <robot xmlns:xacro="http://www.ros.org/wiki/xacro" name="dual_rm_65b_gazebo">
+    <xacro:arg name="gripper_type" default="dummy"/>
     <link name="world"/>
     <joint name="fixed" type="fixed">
@@ -6,5 +7,6 @@
         <child link="base_link_underpan"/>
     </joint>
-    <xacro:include filename="$(find dual_rm_65b_description)/urdf/dual_rm_65b_description.urdf.xacro" />
+    <xacro:arg name="arm_model" default="65b"/>
+    <xacro:include filename="$(find dual_rm_description)/urdf/r2d3_description.urdf.xacro" />
     <gazebo reference="base_link">
         <self_collide>false</self_collide>
@@ -322,4 +324,20 @@
             <state_interface name="velocity"/>
         </joint>
+        <xacro:if value="${'$(arg gripper_type)' == '4c2'}">
+            <joint name="l_gripper_joint">
+                <command_interface name="position"/>
+                <state_interface name="position">
+                    <param name="initial_value">0</param>
+                </state_interface>
+                <state_interface name="velocity"/>
+            </joint>
+            <joint name="r_gripper_joint">
+                <command_interface name="position"/>
+                <state_interface name="position">
+                    <param name="initial_value">0</param>
+                </state_interface>
+                <state_interface name="velocity"/>
+            </joint>
+        </xacro:if>
     </ros2_control>
       <gazebo>

File: ros2_rm_robot/dual_rm_gazebo/config/dual_rm_65b_gz_sim.urdf.xacro (robot description, xacro)
@@ -1,4 +1,5 @@
 <?xml version="1.0"?>
 <robot xmlns:xacro="http://www.ros.org/wiki/xacro" name="dual_rm_65b_gazebo">
+    <xacro:arg name="gripper_type" default="dummy"/>
     <link name="world"/>
     <joint name="fixed" type="fixed">
@@ -6,5 +7,6 @@
         <child link="base_link_underpan"/>
     </joint>
-    <xacro:include filename="$(find dual_rm_65b_description)/urdf/dual_rm_65b_description.urdf.xacro" />
+    <xacro:arg name="arm_model" default="65b"/>
+    <xacro:include filename="$(find dual_rm_description)/urdf/r2d3_description.urdf.xacro" />
     <gazebo reference="base_link">
         <self_collide>false</self_collide>
@@ -322,4 +324,20 @@
             <state_interface name="velocity"/>
         </joint>
+        <xacro:if value="${'$(arg gripper_type)' == '4c2'}">
+            <joint name="l_gripper_joint">
+                <command_interface name="position"/>
+                <state_interface name="position">
+                    <param name="initial_value">0</param>
+                </state_interface>
+                <state_interface name="velocity"/>
+            </joint>
+            <joint name="r_gripper_joint">
+                <command_interface name="position"/>
+                <state_interface name="position">
+                    <param name="initial_value">0</param>
+                </state_interface>
+                <state_interface name="velocity"/>
+            </joint>
+        </xacro:if>
     </ros2_control>
       <gazebo>

File: ros2_rm_robot/dual_rm_gazebo/config/dual_rm_75b_gazebo.urdf.xacro (robot description, xacro)
@@ -1,4 +1,5 @@
 <?xml version="1.0"?>
 <robot xmlns:xacro="http://www.ros.org/wiki/xacro" name="dual_rm_75b_gazebo">
+    <xacro:arg name="gripper_type" default="dummy"/>
     <link name="world"/>
     <joint name="fixed" type="fixed">
@@ -6,5 +7,6 @@
         <child link="base_link_underpan"/>
     </joint>
-    <xacro:include filename="$(find dual_rm_75b_description)/urdf/dual_rm_75b_description.urdf.xacro" />
+    <xacro:arg name="arm_model" default="75b"/>
+    <xacro:include filename="$(find dual_rm_description)/urdf/r2d3_description.urdf.xacro" />
     <gazebo reference="base_link">
         <self_collide>false</self_collide>
@@ -344,4 +346,20 @@
             <state_interface name="velocity"/>
         </joint>
+        <xacro:if value="${'$(arg gripper_type)' == '4c2'}">
+            <joint name="l_gripper_joint">
+                <command_interface name="position"/>
+                <state_interface name="position">
+                    <param name="initial_value">0</param>
+                </state_interface>
+                <state_interface name="velocity"/>
+            </joint>
+            <joint name="r_gripper_joint">
+                <command_interface name="position"/>
+                <state_interface name="position">
+                    <param name="initial_value">0</param>
+                </state_interface>
+                <state_interface name="velocity"/>
+            </joint>
+        </xacro:if>
     </ros2_control>
     <gazebo>

File: ros2_rm_robot/dual_rm_gazebo/config/dual_rm_75b_gz_sim.urdf.xacro (robot description, xacro)
@@ -1,4 +1,5 @@
 <?xml version="1.0"?>
 <robot xmlns:xacro="http://www.ros.org/wiki/xacro" name="dual_rm_75b_gazebo">
+    <xacro:arg name="gripper_type" default="dummy"/>
     <link name="world"/>
     <joint name="fixed" type="fixed">
@@ -6,5 +7,6 @@
         <child link="base_link_underpan"/>
     </joint>
-    <xacro:include filename="$(find dual_rm_75b_description)/urdf/dual_rm_75b_description.urdf.xacro" />
+    <xacro:arg name="arm_model" default="75b"/>
+    <xacro:include filename="$(find dual_rm_description)/urdf/r2d3_description.urdf.xacro" />
     <gazebo reference="base_link">
         <self_collide>false</self_collide>
@@ -344,4 +346,20 @@
             <state_interface name="velocity"/>
         </joint>
+        <xacro:if value="${'$(arg gripper_type)' == '4c2'}">
+            <joint name="l_gripper_joint">
+                <command_interface name="position"/>
+                <state_interface name="position">
+                    <param name="initial_value">0</param>
+                </state_interface>
+                <state_interface name="velocity"/>
+            </joint>
+            <joint name="r_gripper_joint">
+                <command_interface name="position"/>
+                <state_interface name="position">
+                    <param name="initial_value">0</param>
+                </state_interface>
+                <state_interface name="velocity"/>
+            </joint>
+        </xacro:if>
     </ros2_control>
     <gazebo>

Commit message: robot wheels are working in dual_rm_gazebo package

File: ros2_rm_robot/dual_rm_gazebo/config/dual_rm_65b_gazebo.urdf.xacro (robot description, xacro)
@@ -2,9 +2,9 @@
 <robot xmlns:xacro="http://www.ros.org/wiki/xacro" name="dual_rm_65b_gazebo">
     <xacro:arg name="gripper_type" default="dummy"/>
-    <link name="world"/>
+    <!-- <link name="world"/>
     <joint name="fixed" type="fixed">
         <parent link="world"/>
         <child link="base_link_underpan"/>
-    </joint>
+    </joint> -->
     <xacro:arg name="arm_model" default="65b"/>
     <xacro:include filename="$(find dual_rm_description)/urdf/r2d3_description.urdf.xacro" />
@@ -75,49 +75,49 @@
     <gazebo reference="link_right_wheel">
         <self_collide>false</self_collide>
-        <gravity>false</gravity>
+        <!-- <gravity>false</gravity> -->
     </gazebo>
     <gazebo reference="link_left_wheel">
         <self_collide>false</self_collide>
-        <gravity>false</gravity>
+        <!-- <gravity>false</gravity> -->
     </gazebo>
     <gazebo reference="link_swivel_wheel_1_1">
         <self_collide>false</self_collide>
-        <gravity>false</gravity>
+        <!-- <gravity>false</gravity> -->
     </gazebo>
     <gazebo reference="link_swivel_wheel_1_2">
         <self_collide>false</self_collide>
-        <gravity>false</gravity>
+        <!-- <gravity>false</gravity> -->
     </gazebo>
     <gazebo reference="link_swivel_wheel_2_1">
         <self_collide>false</self_collide>
-        <gravity>false</gravity>
+        <!-- <gravity>false</gravity> -->
     </gazebo>
     <gazebo reference="link_swivel_wheel_2_2">
         <self_collide>false</self_collide>
-        <gravity>false</gravity>
+        <!-- <gravity>false</gravity> -->
     </gazebo>
     <gazebo reference="link_swivel_wheel_3_1">
         <self_collide>false</self_collide>
-        <gravity>false</gravity>
+        <!-- <gravity>false</gravity> -->
     </gazebo>
     <gazebo reference="link_swivel_wheel_3_2">
         <self_collide>false</self_collide>
-        <gravity>false</gravity>
+        <!-- <gravity>false</gravity> -->
     </gazebo>
     <gazebo reference="link_swivel_wheel_4_1">
         <self_collide>false</self_collide>
-        <gravity>false</gravity>
+        <!-- <gravity>false</gravity> -->
     </gazebo>
     <gazebo reference="link_swivel_wheel_4_2">
         <self_collide>false</self_collide>
-        <gravity>false</gravity>
+        <!-- <gravity>false</gravity> -->
     </gazebo>
     <gazebo reference="body_base_link">
         <self_collide>false</self_collide>
-        <gravity>false</gravity>
+        <!-- <gravity>false</gravity> -->
     </gazebo>
     <gazebo reference="platform_base_link">
         <self_collide>false</self_collide>
-        <gravity>false</gravity>
+        <!-- <gravity>false</gravity> -->
     </gazebo>
     <gazebo reference="l_base_link1">
@@ -139,8 +139,8 @@
     <gazebo reference="base_link_underpan">
         <self_collide>false</self_collide>
-        <gravity>false</gravity>
+        <!-- <gravity>false</gravity> -->
     </gazebo>
     <gazebo>
-        <is_static>true</is_static>
+        <is_static>false</is_static>
         <self_collide>true</self_collide>
     </gazebo>
@@ -255,5 +255,5 @@
         </joint>
         <joint name="joint_right_wheel">
-            <command_interface name="position"/>
+            <command_interface name="velocity"/>
             <state_interface name="position">
                 <param name="initial_value">0</param>
@@ -262,5 +262,5 @@
         </joint>
         <joint name="joint_left_wheel">
-            <command_interface name="position"/>
+            <command_interface name="velocity"/>
             <state_interface name="position">
                 <param name="initial_value">0</param>

File: ros2_rm_robot/dual_rm_gazebo/config/dual_rm_75b_gazebo.urdf.xacro (robot description, xacro)
@@ -2,9 +2,9 @@
 <robot xmlns:xacro="http://www.ros.org/wiki/xacro" name="dual_rm_75b_gazebo">
     <xacro:arg name="gripper_type" default="dummy"/>
-    <link name="world"/>
+    <!-- <link name="world"/>
     <joint name="fixed" type="fixed">
         <parent link="world"/>
         <child link="base_link_underpan"/>
-    </joint>
+    </joint> -->
     <xacro:arg name="arm_model" default="75b"/>
     <xacro:include filename="$(find dual_rm_description)/urdf/r2d3_description.urdf.xacro" />
@@ -83,49 +83,49 @@
     <gazebo reference="link_right_wheel">
         <self_collide>false</self_collide>
-        <gravity>false</gravity>
+        <!-- <gravity>false</gravity> -->
     </gazebo>
     <gazebo reference="link_left_wheel">
         <self_collide>false</self_collide>
-        <gravity>false</gravity>
+        <!-- <gravity>false</gravity> -->
     </gazebo>
     <gazebo reference="link_swivel_wheel_1_1">
         <self_collide>false</self_collide>
-        <gravity>false</gravity>
+        <!-- <gravity>false</gravity> -->
     </gazebo>
     <gazebo reference="link_swivel_wheel_1_2">
         <self_collide>false</self_collide>
-        <gravity>false</gravity>
+        <!-- <gravity>false</gravity> -->
     </gazebo>
     <gazebo reference="link_swivel_wheel_2_1">
         <self_collide>false</self_collide>
-        <gravity>false</gravity>
+        <!-- <gravity>false</gravity> -->
     </gazebo>
     <gazebo reference="link_swivel_wheel_2_2">
         <self_collide>false</self_collide>
-        <gravity>false</gravity>
+        <!-- <gravity>false</gravity> -->
     </gazebo>
     <gazebo reference="link_swivel_wheel_3_1">
         <self_collide>false</self_collide>
-        <gravity>false</gravity>
+        <!-- <gravity>false</gravity> -->
     </gazebo>
     <gazebo reference="link_swivel_wheel_3_2">
         <self_collide>false</self_collide>
-        <gravity>false</gravity>
+        <!-- <gravity>false</gravity> -->
     </gazebo>
     <gazebo reference="link_swivel_wheel_4_1">
         <self_collide>false</self_collide>
-        <gravity>false</gravity>
+        <!-- <gravity>false</gravity> -->
     </gazebo>
     <gazebo reference="link_swivel_wheel_4_2">
         <self_collide>false</self_collide>
-        <gravity>false</gravity>
+        <!-- <gravity>false</gravity> -->
     </gazebo>
     <gazebo reference="body_base_link">
         <self_collide>false</self_collide>
-        <gravity>false</gravity>
+        <!-- <gravity>false</gravity> -->
     </gazebo>
     <gazebo reference="platform_base_link">
         <self_collide>false</self_collide>
-        <gravity>false</gravity>
+        <!-- <gravity>false</gravity> -->
     </gazebo>
     <gazebo reference="l_base_link1">
@@ -147,8 +147,8 @@
     <gazebo reference="base_link_underpan">
         <self_collide>false</self_collide>
-        <gravity>false</gravity>
+        <!-- <gravity>false</gravity> -->
     </gazebo>
     <gazebo>
-        <is_static>true</is_static>
+        <is_static>false</is_static>
         <self_collide>true</self_collide>
     </gazebo>
@@ -277,5 +277,5 @@
         </joint>
         <joint name="joint_right_wheel">
-            <command_interface name="position"/>
+            <command_interface name="velocity"/>
             <state_interface name="position">
                 <param name="initial_value">0</param>
@@ -284,5 +284,5 @@
         </joint>
         <joint name="joint_left_wheel">
-            <command_interface name="position"/>
+            <command_interface name="velocity"/>
             <state_interface name="position">
                 <param name="initial_value">0</param>
