Commit message: dual_rm_gazebo grippers working with Gripper Action command

File: ros2_rm_robot/dual_rm_description/dual_rm_description/urdf/grippers/4c2_gripper.urdf.xacro (robot description, xacro)
@@ -1,6 +1,7 @@
 <?xml version="1.0" encoding="utf-8"?>
 <robot name="4C2" xmlns:xacro="http://www.ros.org/wiki/xacro">
-  <!-- Default to true so Gazebo apps don't break! -->
+  <!-- Add a specific argument to differentiate between Classic and Harmonic -->
   <xacro:arg name="use_gazebo" default="true"/>
+  <xacro:arg name="gazebo_version" default="classic"/> <!-- 'classic' or 'harmonic' -->
   <xacro:macro name="gripper_4c2" params="prefix parent_link">
   <!-- The joint that actually attaches this gripper to the robot arm -->
@@ -329,9 +330,11 @@
   <ros2_control name="${prefix}Gripper_Hardware" type="system">
     <hardware>
-      <xacro:if value="$(arg use_gazebo)">
+      <xacro:if value="${'$(arg use_gazebo)' == 'true' and '$(arg gazebo_version)' == 'classic'}">
+        <plugin>gazebo_ros2_control/GazeboSystem</plugin>
+      </xacro:if>
+      <xacro:if value="${'$(arg use_gazebo)' == 'true' and '$(arg gazebo_version)' == 'harmonic'}">
         <plugin>gz_ros2_control/GazeboSimSystem</plugin>
       </xacro:if>
       <xacro:unless value="$(arg use_gazebo)">
-        <!-- Use a mock system to prevent MuJoCo from spawning multiple physics instances -->
         <plugin>mock_components/GenericSystem</plugin>
       </xacro:unless>
@@ -390,4 +393,39 @@
     </joint>
   </ros2_control>
+  <!-- ═══════════════════════════════════════════════════════════
+       GAZEBO SPECIFIC: Mimic Joint Plugins
+       ═══════════════════════════════════════════════════════════ -->
+  <gazebo>
+    <plugin name="${prefix}mimic_r3" filename="libroboticsgroup_upatras_gazebo_mimic_joint_plugin.so">
+      <joint>${prefix}gripper_joint</joint>
+      <mimicJoint>${prefix}r_3_joint</mimicJoint>
+      <multiplier>1.0</multiplier>
+      <maxEffort>0.5</maxEffort>
+    </plugin>
+    <plugin name="${prefix}mimic_l1" filename="libroboticsgroup_upatras_gazebo_mimic_joint_plugin.so">
+      <joint>${prefix}gripper_joint</joint>
+      <mimicJoint>${prefix}l_1_joint</mimicJoint>
+      <multiplier>1.0</multiplier>
+      <maxEffort>0.5</maxEffort>
+    </plugin>
+    <plugin name="${prefix}mimic_l3" filename="libroboticsgroup_upatras_gazebo_mimic_joint_plugin.so">
+      <joint>${prefix}gripper_joint</joint>
+      <mimicJoint>${prefix}l_3_joint</mimicJoint>
+      <multiplier>1.0</multiplier>
+      <maxEffort>0.5</maxEffort>
+    </plugin>
+    <plugin name="${prefix}mimic_r2" filename="libroboticsgroup_upatras_gazebo_mimic_joint_plugin.so">
+      <joint>${prefix}gripper_joint</joint>
+      <mimicJoint>${prefix}r_2_joint</mimicJoint>
+      <multiplier>1.0</multiplier>
+      <maxEffort>0.5</maxEffort>
+    </plugin>
+    <plugin name="${prefix}mimic_l2" filename="libroboticsgroup_upatras_gazebo_mimic_joint_plugin.so">
+      <joint>${prefix}gripper_joint</joint>
+      <mimicJoint>${prefix}l_2_joint</mimicJoint>
+      <multiplier>1.0</multiplier>
+      <maxEffort>0.5</maxEffort>
+    </plugin>
+  </gazebo>
   </xacro:macro>
 </robot>

File: ros2_rm_robot/dual_rm_gazebo/config/dual_rm_65b_gazebo.urdf.xacro (robot description, xacro)
@@ -324,5 +324,6 @@
             <state_interface name="velocity"/>
         </joint>
-        <xacro:if value="${'$(arg gripper_type)' == '4c2'}">
+        <!-- The control is defined in src/ros2_rm_robot/dual_rm_description/dual_rm_description/urdf/grippers/4c2_gripper.urdf.xacro -->
+        <!-- <xacro:if value="${'$(arg gripper_type)' == '4c2'}">
             <joint name="l_gripper_joint">
                 <command_interface name="position"/>
@@ -339,5 +340,5 @@
                 <state_interface name="velocity"/>
             </joint>
-        </xacro:if>
+        </xacro:if> -->
     </ros2_control>
       <gazebo>

File: ros2_rm_robot/dual_rm_gazebo/config/dual_rm_75b_gazebo.urdf.xacro (robot description, xacro)
@@ -346,5 +346,6 @@
             <state_interface name="velocity"/>
         </joint>
-        <xacro:if value="${'$(arg gripper_type)' == '4c2'}">
+        <!-- The control is defined in src/ros2_rm_robot/dual_rm_description/dual_rm_description/urdf/grippers/4c2_gripper.urdf.xacro -->
+        <!-- <xacro:if value="${'$(arg gripper_type)' == '4c2'}">
             <joint name="l_gripper_joint">
                 <command_interface name="position"/>
@@ -361,5 +362,5 @@
                 <state_interface name="velocity"/>
             </joint>
-        </xacro:if>
+        </xacro:if> -->
     </ros2_control>
     <gazebo>

Commit message: fixed gripper joint not found in r2d3_apps bringup due to change in 4c2 xacro

File: ros2_rm_robot/dual_rm_description/dual_rm_description/urdf/grippers/4c2_gripper.urdf.xacro (robot description, xacro)
@@ -3,5 +3,5 @@
   <!-- Add a specific argument to differentiate between Classic and Harmonic -->
   <xacro:arg name="use_gazebo" default="true"/>
-  <xacro:arg name="gazebo_version" default="classic"/> <!-- 'classic' or 'harmonic' -->
+  <xacro:arg name="gazebo_version" default="$(optenv GAZEBO_VERSION classic)"/>
   <xacro:macro name="gripper_4c2" params="prefix parent_link">
   <!-- The joint that actually attaches this gripper to the robot arm -->
@@ -394,38 +394,40 @@
   </ros2_control>
   <!-- ═══════════════════════════════════════════════════════════
-       GAZEBO SPECIFIC: Mimic Joint Plugins
+       GAZEBO SPECIFIC: Mimic Joint Plugins (Classic only)
        ═══════════════════════════════════════════════════════════ -->
-  <gazebo>
-    <plugin name="${prefix}mimic_r3" filename="libroboticsgroup_upatras_gazebo_mimic_joint_plugin.so">
-      <joint>${prefix}gripper_joint</joint>
-      <mimicJoint>${prefix}r_3_joint</mimicJoint>
-      <multiplier>1.0</multiplier>
-      <maxEffort>0.5</maxEffort>
-    </plugin>
-    <plugin name="${prefix}mimic_l1" filename="libroboticsgroup_upatras_gazebo_mimic_joint_plugin.so">
-      <joint>${prefix}gripper_joint</joint>
-      <mimicJoint>${prefix}l_1_joint</mimicJoint>
-      <multiplier>1.0</multiplier>
-      <maxEffort>0.5</maxEffort>
-    </plugin>
-    <plugin name="${prefix}mimic_l3" filename="libroboticsgroup_upatras_gazebo_mimic_joint_plugin.so">
-      <joint>${prefix}gripper_joint</joint>
-      <mimicJoint>${prefix}l_3_joint</mimicJoint>
-      <multiplier>1.0</multiplier>
-      <maxEffort>0.5</maxEffort>
-    </plugin>
-    <plugin name="${prefix}mimic_r2" filename="libroboticsgroup_upatras_gazebo_mimic_joint_plugin.so">
-      <joint>${prefix}gripper_joint</joint>
-      <mimicJoint>${prefix}r_2_joint</mimicJoint>
-      <multiplier>1.0</multiplier>
-      <maxEffort>0.5</maxEffort>
-    </plugin>
-    <plugin name="${prefix}mimic_l2" filename="libroboticsgroup_upatras_gazebo_mimic_joint_plugin.so">
-      <joint>${prefix}gripper_joint</joint>
-      <mimicJoint>${prefix}l_2_joint</mimicJoint>
-      <multiplier>1.0</multiplier>
-      <maxEffort>0.5</maxEffort>
-    </plugin>
-  </gazebo>
+  <xacro:if value="${'$(arg use_gazebo)' == 'true' and '$(arg gazebo_version)' == 'classic'}">
+    <gazebo>
+      <plugin name="${prefix}mimic_r3" filename="libroboticsgroup_upatras_gazebo_mimic_joint_plugin.so">
+        <joint>${prefix}gripper_joint</joint>
+        <mimicJoint>${prefix}r_3_joint</mimicJoint>
+        <multiplier>1.0</multiplier>
+        <maxEffort>0.5</maxEffort>
+      </plugin>
+      <plugin name="${prefix}mimic_l1" filename="libroboticsgroup_upatras_gazebo_mimic_joint_plugin.so">
+        <joint>${prefix}gripper_joint</joint>
+        <mimicJoint>${prefix}l_1_joint</mimicJoint>
+        <multiplier>1.0</multiplier>
+        <maxEffort>0.5</maxEffort>
+      </plugin>
+      <plugin name="${prefix}mimic_l3" filename="libroboticsgroup_upatras_gazebo_mimic_joint_plugin.so">
+        <joint>${prefix}gripper_joint</joint>
+        <mimicJoint>${prefix}l_3_joint</mimicJoint>
+        <multiplier>1.0</multiplier>
+        <maxEffort>0.5</maxEffort>
+      </plugin>
+      <plugin name="${prefix}mimic_r2" filename="libroboticsgroup_upatras_gazebo_mimic_joint_plugin.so">
+        <joint>${prefix}gripper_joint</joint>
+        <mimicJoint>${prefix}r_2_joint</mimicJoint>
+        <multiplier>1.0</multiplier>
+        <maxEffort>0.5</maxEffort>
+      </plugin>
+      <plugin name="${prefix}mimic_l2" filename="libroboticsgroup_upatras_gazebo_mimic_joint_plugin.so">
+        <joint>${prefix}gripper_joint</joint>
+        <mimicJoint>${prefix}l_2_joint</mimicJoint>
+        <multiplier>1.0</multiplier>
+        <maxEffort>0.5</maxEffort>
+      </plugin>
+    </gazebo>
+  </xacro:if>
   </xacro:macro>
 </robot>

File: ros2_rm_robot/dual_rm_gazebo/config/dual_rm_65b_gz_sim.urdf.xacro (robot description, xacro)
@@ -2,14 +2,14 @@
 <robot xmlns:xacro="http://www.ros.org/wiki/xacro" name="dual_rm_65b_gazebo">
     <xacro:arg name="gripper_type" default="dummy"/>
-    <link name="world"/>
+    <!-- <link name="world"/>
     <joint name="fixed" type="fixed">
         <parent link="world"/>
         <child link="base_link_underpan"/>
-    </joint>
+    </joint> -->
     <xacro:arg name="arm_model" default="65b"/>
     <xacro:include filename="$(find dual_rm_description)/urdf/r2d3_description.urdf.xacro" />
     <gazebo reference="base_link">
         <self_collide>false</self_collide>
-        <gravity>false</gravity>
+        <!-- <gravity>false</gravity> -->
     </gazebo>
     <gazebo reference="r_link1">
@@ -75,49 +75,49 @@
     <gazebo reference="link_right_wheel">
         <self_collide>false</self_collide>
-        <gravity>false</gravity>
+        <!-- <gravity>false</gravity> -->
     </gazebo>
     <gazebo reference="link_left_wheel">
         <self_collide>false</self_collide>
-        <gravity>false</gravity>
+        <!-- <gravity>false</gravity> -->
     </gazebo>
     <gazebo reference="link_swivel_wheel_1_1">
         <self_collide>false</self_collide>
-        <gravity>false</gravity>
+        <!-- <gravity>false</gravity> -->
     </gazebo>
     <gazebo reference="link_swivel_wheel_1_2">
         <self_collide>false</self_collide>
-        <gravity>false</gravity>
+        <!-- <gravity>false</gravity> -->
     </gazebo>
     <gazebo reference="link_swivel_wheel_2_1">
         <self_collide>false</self_collide>
-        <gravity>false</gravity>
+        <!-- <gravity>false</gravity> -->
     </gazebo>
     <gazebo reference="link_swivel_wheel_2_2">
         <self_collide>false</self_collide>
-        <gravity>false</gravity>
+        <!-- <gravity>false</gravity> -->
     </gazebo>
     <gazebo reference="link_swivel_wheel_3_1">
         <self_collide>false</self_collide>
-        <gravity>false</gravity>
+        <!-- <gravity>false</gravity> -->
     </gazebo>
     <gazebo reference="link_swivel_wheel_3_2">
         <self_collide>false</self_collide>
-        <gravity>false</gravity>
+        <!-- <gravity>false</gravity> -->
     </gazebo>
     <gazebo reference="link_swivel_wheel_4_1">
         <self_collide>false</self_collide>
-        <gravity>false</gravity>
+        <!-- <gravity>false</gravity> -->
     </gazebo>
     <gazebo reference="link_swivel_wheel_4_2">
         <self_collide>false</self_collide>
-        <gravity>false</gravity>
+        <!-- <gravity>false</gravity> -->
     </gazebo>
     <gazebo reference="body_base_link">
         <self_collide>false</self_collide>
-        <gravity>false</gravity>
+        <!-- <gravity>false</gravity> -->
     </gazebo>
     <gazebo reference="platform_base_link">
         <self_collide>false</self_collide>
-        <gravity>false</gravity>
+        <!-- <gravity>false</gravity> -->
     </gazebo>
     <gazebo reference="l_base_link1">
@@ -139,8 +139,8 @@
     <gazebo reference="base_link_underpan">
         <self_collide>false</self_collide>
-        <gravity>false</gravity>
+        <!-- <gravity>false</gravity> -->
     </gazebo>
     <gazebo>
-        <is_static>true</is_static>
+        <is_static>false</is_static>
         <self_collide>true</self_collide>
     </gazebo>
@@ -255,5 +255,5 @@
         </joint>
         <joint name="joint_right_wheel">
-            <command_interface name="position"/>
+            <command_interface name="velocity"/>
             <state_interface name="position">
                 <param name="initial_value">0</param>
@@ -262,5 +262,5 @@
         </joint>
         <joint name="joint_left_wheel">
-            <command_interface name="position"/>
+            <command_interface name="velocity"/>
             <state_interface name="position">
                 <param name="initial_value">0</param>
@@ -324,5 +324,5 @@
             <state_interface name="velocity"/>
         </joint>
-        <xacro:if value="${'$(arg gripper_type)' == '4c2'}">
+        <!-- <xacro:if value="${'$(arg gripper_type)' == '4c2'}">
             <joint name="l_gripper_joint">
                 <command_interface name="position"/>
@@ -339,5 +339,5 @@
                 <state_interface name="velocity"/>
             </joint>
-        </xacro:if>
+        </xacro:if> -->
     </ros2_control>
       <gazebo>
