Commit message: fixed wrong moveemnt of grippers in dual_rm_gazebo package

File: ros2_rm_robot/dual_rm_description/dual_rm_description/urdf/r2d3_description.urdf.xacro (robot description, xacro)
@@ -5,4 +5,6 @@
     <xacro:arg name="gripper_type" default="$(optenv GRIPPER_TYPE dummy)"/>
     <xacro:property name="gripper_type" value="$(arg gripper_type)"/>
+    <xacro:arg name="gz_sim_gripper_path" default=""/>
+    <xacro:property name="gz_sim_gripper_path" value="$(arg gz_sim_gripper_path)"/>
     <!-- ═══════════════════════════════════════════════════════════
          Shared components (identical for both arm variants)
@@ -27,6 +29,11 @@
     </xacro:if>
     <xacro:if value="${gripper_type == '4c2'}">
-        <!-- Load the new 4c2 Gripper Macro -->
-        <xacro:include filename="$(find dual_rm_description)/urdf/grippers/4c2_gripper.urdf.xacro"/>
+        <!-- Dynamic Routing: Inject specialized gz_sim file if provided, else default to Classic -->
+        <xacro:if value="${gz_sim_gripper_path != ''}">
+            <xacro:include filename="${gz_sim_gripper_path}"/>
+        </xacro:if>
+        <xacro:if value="${gz_sim_gripper_path == ''}">
+            <xacro:include filename="$(find dual_rm_description)/urdf/grippers/4c2_gripper.urdf.xacro"/>
+        </xacro:if>
         <!-- Attach to the 6th link for the 65b model -->
         <xacro:if value="${arm_model == '65b'}">

File: ros2_rm_robot/dual_rm_gazebo/config/dual_rm_65b_gz_sim.urdf.xacro (robot description, xacro)
@@ -143,5 +143,5 @@
     <gazebo>
         <is_static>false</is_static>
-        <self_collide>true</self_collide>
+        <self_collide>false</self_collide>
     </gazebo>
     <ros2_control name="GazeboSystem" type="system">

File: ros2_rm_robot/dual_rm_gazebo/config/dual_rm_75b_gz_sim.urdf.xacro (robot description, xacro)
@@ -151,5 +151,5 @@
     <gazebo>
         <is_static>true</is_static>
-        <self_collide>true</self_collide>
+        <self_collide>false</self_collide>
     </gazebo>
     <ros2_control name="GazeboSystem" type="system">
@@ -277,5 +277,5 @@
         </joint>
         <joint name="joint_right_wheel">
-            <command_interface name="position"/>
+            <command_interface name="velocity"/>
             <state_interface name="position">
                 <param name="initial_value">0</param>
@@ -284,5 +284,5 @@
         </joint>
         <joint name="joint_left_wheel">
-            <command_interface name="position"/>
+            <command_interface name="velocity"/>
             <state_interface name="position">
                 <param name="initial_value">0</param>
@@ -346,5 +346,5 @@
             <state_interface name="velocity"/>
         </joint>
-        <xacro:if value="${'$(arg gripper_type)' == '4c2'}">
+        <!-- <xacro:if value="${'$(arg gripper_type)' == '4c2'}">
             <joint name="l_gripper_joint">
                 <command_interface name="position"/>
@@ -361,5 +361,5 @@
                 <state_interface name="velocity"/>
             </joint>
-        </xacro:if>
+        </xacro:if> -->
     </ros2_control>
     <gazebo>
